File: Masochist.kicad_pcb (KiCad board)
At the start: 2 copper layers, 114.3 x 58.7 mm, 51 parts, among them J1 USB_C_Receptacle_USB2.0, SW1 SW_Push, U1 ATmega32U4-MU, U2 USBLC6-2SC6, Y1 16 MHz

Commit message: add silkscreen and distribution credits
Parts:
- moved D11 3.97 mm to (93.7, 163.5)
Routing:
- net Row2: track 128.0 -> 131.2 mm
- net Net-(D11-Pad2): track 8.05 -> 8.87 mm
Other:
- board text added: "Distributed by Kiser Designs"
- board text added: "Silkscreen by killwhiteyy"
- board text removed: "SUFFER."
Changed lines of the file:
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@@
   )
   (footprint "Diode_SMD:D_SOD-123" (layer "B.Cu")
-    (at 91.28125 166.6875 90)
+    (at 93.6625 163.5125 90)
     (descr "SOD-123")
     (tags "SOD-123")
@@
   (gr_arc (start 77.7875 115.8875) (mid 78.019984 115.326234) (end 78.58125 115.09375) (layer "Edge.Cuts") (width 0.05))
   (gr_line (start 77.7875 115.8875) (end 77.7875 116.68125) (layer "Edge.Cuts") (width 0.05))
+  (gr_text "Silkscreen by killwhiteyy" (at 45.24375 170.65625) (layer "B.SilkS")
+    (effects (font (size 1.5 1.5) (thickness 0.3)) (justify mirror))
+  )
   (gr_text "Made with <3 by Zicodia" (at 121.44375 170.65625) (layer "B.SilkS")
     (effects (font (size 1.5 1.5) (thickness 0.3)) (justify mirror))
   )
-  (gr_text "SUFFER." (at 83.34375 147.6375) (layer "F.SilkS")
-    (effects (font (size 50.000002 15) (thickness 3.75)))
+  (gr_text "Distributed by\nKiser Designs" (at 83.34375 170.65625) (layer "B.SilkS")
+    (effects (font (size 1.5 1.5) (thickness 0.3)) (justify mirror))
   )
   (segment (start 119.29576 150.188582) (end 118.936427 149.829249) (width 0.254) (layer "B.Cu") (net 1))
@@
   (segment (start 137.84 161.408538) (end 124.862712 148.43125) (width 0.254) (layer "B.Cu") (net 4))
   (segment (start 115.998489 146.910989) (end 115.25625 146.16875) (width 0.254) (layer "B.Cu") (net 4))
-  (segment (start 123.03125 168.3375) (end 43.65625 168.3375) (width 0.254) (layer "B.Cu") (net 4))
+  (segment (start 93.648122 168.3375) (end 43.65625 168.3375) (width 0.254) (layer "B.Cu") (net 4))
+  (segment (start 93.6625 168.323122) (end 93.648122 168.3375) (width 0.254) (layer "B.Cu") (net 4))
   (segment (start 137.84 164.86) (end 137.84 161.408538) (width 0.254) (layer "B.Cu") (net 4))
   (segment (start 116.614011 147.336568) (end 116.188432 146.910989) (width 0.254) (layer "B.Cu") (net 4))
   (segment (start 120.006568 147.336568) (end 116.614011 147.336568) (width 0.254) (layer "B.Cu") (net 4))
+  (segment (start 93.6625 165.1625) (end 93.6625 168.323122) (width 0.254) (layer "B.Cu") (net 4))
+  (segment (start 123.03125 168.3375) (end 93.648122 168.3375) (width 0.254) (layer "B.Cu") (net 4))
   (segment (start 123.03125 168.3375) (end 134.3625 168.3375) (width 0.254) (layer "B.Cu") (net 4))
   (segment (start 134.3625 168.3375) (end 137.84 164.86) (width 0.254) (layer "B.Cu") (net 4))
@@
   (segment (start 100.80625 126.52375) (end 100.80625 126.9375) (width 0.254) (layer "B.Cu") (net 26))
   (segment (start 95.40875 121.12625) (end 100.80625 126.52375) (width 0.254) (layer "B.Cu") (net 26))
-  (segment (start 91.28125 164.62375) (end 91.28125 165.0375) (width 0.254) (layer "B.Cu") (net 27))
-  (segment (start 85.88375 159.22625) (end 91.28125 164.62375) (width 0.254) (layer "B.Cu") (net 27))
+  (segment (start 88.52 161.8625) (end 93.6625 161.8625) (width 0.254) (layer "B.Cu") (net 27))
+  (segment (start 85.88375 159.22625) (end 88.52 161.8625) (width 0.254) (layer "B.Cu") (net 27))
   (segment (start 86.51875 145.57375) (end 86.51875 145.9875) (width 0.254) (layer "B.Cu") (net 28))
   (segment (start 81.12125 140.17625) (end 86.51875 145.57375) (width 0.254) (layer "B.Cu") (net 28))

Commit message: add production files
Parts:
- added ?: , , F.Cu at (45.2, 121.4)
- added G***: LOGO, LOGO, F.Cu at (83.3, 145.3)
- added G***: LOGO, LOGO, B.Cu at (83.3, 145.3)
- added REF**: MountingHole_2.2mm_M2_Pad, cftkb:MountingHole_2.2mm_M2_Pad, F.Cu at (121.4, 121.4)
- added REF**: MountingHole_2.2mm_M2_Pad, cftkb:MountingHole_2.2mm_M2_Pad, F.Cu at (45.2, 159.5)
- added REF**: MountingHole_2.2mm_M2_Pad, cftkb:MountingHole_2.2mm_M2_Pad, F.Cu at (121.4, 159.5)
Routing:
- net +5V: track 134.6 -> 123.5 mm, vias 11 -> 10
- net GND: track 100.5 -> 104.7 mm, vias 2 -> 15
- net Col5: track 60.8 -> 62.0 mm
- net XTAL2: track 13.5 -> 14.5 mm
